File: meterbar.kicad_pcb (KiCad board)
At the start: 2 copper layers, 46 parts, among them J1 Screw_Terminal_01x02, J2 Screw_Terminal_01x03, J3 40HAT, J4 Screw_Terminal_01x02, J5 Conn_02x08_Odd_Even, Q1 DMC2053UVT, Q2 DMC2053UVT, Q3 DMC2053UVT, Q4 DMC2053UVT, Q5 DMC2053UVT, U1 LM1085-3.3, U2 AD5360BSTZ, U3 ADR02AR

Commit message: ready to order
Routing:
- net GND: track 24.5 -> 29.8 mm
- net +3V3: track 15.7 -> 20.7 mm
Other:
- board outline added: 56 x 85 mm
- board text added: "bot"
- board text added: "top"
- board text added: "vu meter bar v1.0"
